Commit message: assd

File: hw5code/urdf/robot.urdf (robot description, URDF)
Before this commit: robot robot, 19 links, 18 joints
Joints:
- removed joint Dwarfs/Doc
- removed joint Dwarfs/Grumpy
- removed joint Dwarfs/Sleepy
- added joint Photon/1: type continuous, parent motor2base, child motor2output, axis 0 0 1
- added joint Photon/5: type continuous, parent motor0base, child motor0output, axis 0 0 1
- added joint Photon/6: type continuous, parent motor1base, child motor1output, axis 0 0 1

Commit message: asdas

File: hw5code/urdf/robot.urdf (robot description, URDF)
Before this commit: robot robot, 19 links, 18 joints
Joints:
- joint connect-motor1output-motor2base: origin xyz=0.5 0 0.036 rpy=0 0 0 -> xyz=0.3 0 0.036 rpy=0 0 0
- joint connect-motor2output-tip: origin xyz=0.5 0 0.0335 rpy=0 1.57 0 -> xyz=0.3 0 0.0335 rpy=0 1.57 0

Commit message: asdas

File: hw5code/urdf/robot.urdf (robot description, URDF)
Before this commit: robot robot, 19 links, 18 joints
Links:
- link link1part1: geometry visual box size=0.03 0.08 0.005
- link link2: geometry visual box size=0.3 0.05 0.005
- link link3: geometry visual box size=0.3 0.05 0.005

Commit message: asdas

File: hw5code/urdf/robot.urdf (robot description, URDF)
Before this commit: robot robot, 19 links, 18 joints
Joints:
- joint connect-motor2output-tip: origin xyz=0.3 0 0.0335 rpy=0 1.57 0 -> xyz=0.0 0 0.0335 rpy=0 1.57 0

Commit message: asdas

File: hw5code/urdf/robot.urdf (robot description, URDF)
Before this commit: robot robot, 19 links, 18 joints
Joints:
- joint connect-motor2output-tip: origin xyz=0.0 0 0.0335 rpy=0 1.57 0 -> xyz=0.3 0 0.0335 rpy=0 1.57 0

Commit message: asds

File: hw5code/urdf/robot.urdf (robot description, URDF)
Before this commit: robot robot, 19 links, 18 joints
Joints:
- joint connect-motor2output-tip: origin xyz=0.3 0 0.0335 rpy=0 1.57 0 -> xyz=0 0 0
